File: lcd-square-4-4848/usb_power.kicad_sch (KiCad schematic)
At the start: 5 parts, among them J4 USB_C_Receptacle_USB2.0_16P

Commit message: Slight changes
Parts:
- C8: JLCPCB Part # (none) -> C1779
- C9: footprint Capacitor_SMD:C_0603_1608Metric -> Capacitor_SMD:C_0402_1005Metric; JLCPCB Part # (none) -> C307331
- J4: JLCPCB Part # (none) -> C963412
- R10, R9: JLCPCB Part # (none) -> C25905
Changed lines of the file:
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@@
+			)
+		)
+		(property "JLCPCB Part #" "C1779"
+			(at 162.56 60.96 0)
+			(effects
+				(font
+					(size 1.27 1.27)
+				)
+				(hide yes)
 			)
 		)
@@
 			)
 		)
+		(property "JLCPCB Part #" "C25905"
+			(at 180.34 76.2 0)
+			(effects
+				(font
+					(size 1.27 1.27)
+				)
+				(hide yes)
+			)
+		)
 		(pin "2"
 		)
@@
 			)
 		)
-		(property "Footprint" "Capacitor_SMD:C_0603_1608Metric"
+		(property "Footprint" "Capacitor_SMD:C_0402_1005Metric"
 			(at 172.72 60.96 0)
 			(effects
@@
 		)
 		(property "Description" "Unpolarized capacitor, small symbol"
+			(at 172.72 60.96 0)
+			(effects
+				(font
+					(size 1.27 1.27)
+				)
+				(hide yes)
+			)
+		)
+		(property "JLCPCB Part #" "C307331"
 			(at 172.72 60.96 0)
 			(effects
@@
 			)
 		)
+		(property "JLCPCB Part #" "C25905"
+			(at 180.34 78.74 0)
+			(effects
+				(font
+					(size 1.27 1.27)
+				)
+				(hide yes)
+			)
+		)
 		(pin "2"
 		)
@@
 			(at 203.2 86.36 0)
 			(effects
+				(font
+					(size 1.27 1.27)
+				)
+				(hide yes)
+			)
+		)
+		(property "JLCPCB Part #" "C963412 "
+			(at 203.2 86.36 0)
+			(effects
