File: lcd-square-4inch/lcd-square-4inch.kicad_sch (KiCad schematic)
At the start: 42 parts, among them J1 Conn_01x02_MountingPin, J2 Micro_SD_Card_Det1, J3 Conn_01x30_MountingPin, J4 SWD, J5 Conn_01x40_MountingPin, U1 MAX98357A, U2 TPS61169

Commit message: Add QSPI Flash trace length matching to 5 inch LCD
Parts:
- H1, H2, H3, H4: JLCPCB Part # (none) -> C2915636; now in the parts list
